File: hardware/SuperCap_Ctrl/SuperCap_Ctrl.kicad_pcb (KiCad board)
At the start: 2 copper layers, 45 x 45 mm, 89 parts, among them J1 Conn_01x02, J2 Conn_01x04, J3 Conn_01x32_MountingPin, J4 Conn_01x03, Q1 Si2308, Q3 Si2308, Q4 Si2308, Q5 Si2308, Q6 Si2308, U1 STM32G474VCTx, U4 TJA1044GT/3Z, U5 XC6206PxxxMR, U8 XC6206PxxxMR, X1 CSTCE24M

Commit message: RMUC version
Parts:
- R26: value 33R -> 51R
Connections:
- U4 pad 5: unconnected-(U4-VIO-Pad5) -> +3.3V
Routing:
- net +3.3V: track 141.6 -> 150.6 mm, vias 15 -> 17
Other:
- board text added: "WEILAI_SuperCap_Ctrl_v0.3"
- board text removed: "WEILAI_SuperCap_Ctrl_v0.2"
