File: hardware/SuperCap_Ctrl/SuperCap_Ctrl.kicad_sch (KiCad schematic)
At the start: 87 parts, among them J1 Conn_01x02, J2 Conn_01x04, J3 Conn_01x32_MountingPin, J4 Conn_01x03, Q1 Si2308, Q3 Si2308, Q4 Si2308, Q5 Si2308, Q6 Si2308, U1 STM32G474VCTx, U4 TJA1044GT/3Z, U5 XC6206PxxxMR, U8 XC6206PxxxMR, X1 CSTCE24M

Commit message: RMUC version
Connections:
- net +3.3V: now also U4.5 (VIO)
- net GND: now also R10.1, R7.1, R8.1, R9.1; no longer Q3.2 (D), Q4.2 (D), Q5.2 (D), Q6.2 (D)
- net at Q6.3 (S): now also D7.3 (K1); no longer R10.1
- net at R10.2: now also Q6.2 (D); no longer D7.3 (K1)
- net at Q3.3 (S): now also D6.4 (K2); no longer R7.1
- net at R7.2: now also Q3.2 (D); no longer D6.4 (K2)
- net at Q4.3 (S): now also D6.3 (K1); no longer R8.1
- net at Q5.3 (S): now also D7.4 (K2); no longer R9.1
- net at R9.2: now also Q5.2 (D); no longer D7.4 (K2)
- net at R8.2: now also Q4.2 (D); no longer D6.3 (K1)
- no-connect marks 54 -> 53
Other:
- moved on the sheet: D6, D7, FB6, FB7, Q3, Q4, Q5, Q6, R10, R7, R8, R9
